Commit message: Remove mimic joints.

File: robot_specific_config/abb_irb6640_support/urdf/irb6640_205/irb6640_205_macro.ros2_control.xacro (robot description, xacro)
@@ -93,5 +93,5 @@
       </joint>
       <!-- Mimic joints -->
-      <joint name="${prefix}piston_joint">
+      <!-- <joint name="${prefix}piston_joint">
         <param name="mimic">joint_2</param>
         <param name="multiplier">-1.3</param>
@@ -104,5 +104,5 @@
         <command_interface name="position"/>
         <state_interface name="position"/>
-      </joint>
+      </joint> -->
     </ros2_control>
     <xacro:if value="$(arg sim_gazebo_classic)">
