Commit message: Update irb6640_205_macro.xacro
Fix joint 5 limits

File: robot_specific_config/abb_irb6640_support/urdf/irb6640_205/irb6640_205_macro.xacro (robot description, xacro)
@@ -227,5 +227,5 @@
       <child link="${prefix}link5" />
       <axis xyz="0 1 0" />
-      <limit effort="0" lower="${radians(-100)}" upper="${radians(100)}" velocity="${radians(120)}" />
+      <limit effort="0" lower="${radians(-120)}" upper="${radians(120)}" velocity="${radians(120)}" />
     </joint>
     <!-- joint 6 -->
